File: peripherals.kicad_sch (KiCad schematic)
At the start: 58 parts, among them J801 Socket_Samtec_ERF5_2x20_ERF5-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, J802 JST_SH_1x4_SM04B-SRSS-TB-LF-SN, J803 JST_SH_1x4_SM04B-SRSS-TB-LF-SN, J804 JST_SH_1x2_SM02B-SRSS-TB-LF-SN, U801 PN7160A1_VFQFN, Y801 Resonator_27.12MHz_XRCGB

Commit message: [#58133] Update from lib
Parts:
- R801, R803, R805: now in the parts list
- Y801: footprint antmicro-footprints:Oscillator_SMD_ECS_2016MV_2x1.6x0.85mm -> antmicro-footprints:Resonator_SMD_Murata_XRCGB_2x1.6x0.65mm
Connections:
- net GND: now also J802.MP, J803.MP, J804.MP; no longer J802.SH1, J802.SH2, J803.SH1, J803.SH2, J804.SH1, J804.SH2
Changed lines of the file:
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@@
   (junction (at 41.91 179.07) (diameter 0) (color 0 0 0 0)
   )
-  (junction (at 106.68 102.87) (diameter 0) (color 0 0 0 0)
-  )
   (junction (at 309.88 158.75) (diameter 0) (color 0 0 0 0)
   )
   (junction (at 320.04 158.75) (diameter 0) (color 0 0 0 0)
   )
-  (junction (at 374.65 111.76) (diameter 0) (color 0 0 0 0)
-  )
-  (junction (at 106.68 40.64) (diameter 0) (color 0 0 0 0)
-  )
   (junction (at 314.96 166.37) (diameter 0) (color 0 0 0 0)
   )
@@
     (stroke (width 0) (type default))
   )
-  (wire (pts (xy 109.22 100.33) (xy 106.68 100.33))
-    (stroke (width 0) (type default))
-  )
   (bus (pts (xy 24.13 209.55) (xy 24.13 212.09))
     (stroke (width 0) (type default))
@@
     (stroke (width 0) (type default))
   )
-  (wire (pts (xy 374.65 111.76) (xy 374.65 109.22))
-    (stroke (width 0) (type default))
-  )
   (bus (pts (xy 111.76 185.42) (xy 111.76 187.96))
     (stroke (width 0) (type default))
@@
     (stroke (width 0) (type default))
   )
-  (wire (pts (xy 374.65 109.22) (xy 375.92 109.22))
-    (stroke (width 0) (type default))
-  )
   (bus (pts (xy 24.13 168.91) (xy 24.13 179.07))
     (stroke (width 0) (type default))
@@
     (stroke (width 0) (type default))
   )
-  (wire (pts (xy 106.68 100.33) (xy 106.68 102.87))
-    (stroke (width 0) (type default))
-  )
   (wire (pts (xy 55.88 222.25) (xy 73.66 222.25))
     (stroke (width 0) (type default))
@@
     (stroke (width 0) (type default))
   )
-  (wire (pts (xy 106.68 38.1) (xy 106.68 40.64))
-    (stroke (width 0) (type default))
-  )
   (wire (pts (xy 236.22 114.3) (xy 236.22 115.57))
     (stroke (width 0) (type default))
@@
     (stroke (width 0.3) (type solid))
   )
-  (wire (pts (xy 109.22 38.1) (xy 106.68 38.1))
-    (stroke (width 0) (type default))
-  )
   (image (at 71.628 271.526) (scale 0.15)
     (data
@@
     (pin "3")
     (pin "4")
-    (pin "SH1")
-    (pin "SH2")
+    (pin "MP")
     (instances
       (project "cm4-baseboard"
@@
   )
   (symbol (lib_id "antmicroResistors0402:R_10k_0402") (at 236.22 120.65 90) (unit 1)
-    (in_bom no) (on_board yes) (dnp yes)
+    (in_bom yes) (on_board yes) (dnp yes)
     (property "Reference" "R803" (at 237.49 116.84 90)
       (effects (font (size 1.27 1.27) (thickness 0.15)) (justify right))
@@
       (effects (font (size 1.27 1.27) (thickness 0.15)) (justify left bottom) hide)
     )
-    (property "Footprint" "antmicro-footprints:Oscillator_SMD_ECS_2016MV_2x1.6x0.85mm" (at 334.01 168.91 0)
+    (property "Footprint" "antmicro-footprints:Resonator_SMD_Murata_XRCGB_2x1.6x0.65mm" (at 334.01 168.91 0)
       (effects (font (size 1.27 1.27) (thickness 0.15)) (justify left bottom) hide)
     )
@@
   )
   (symbol (lib_id "antmicroResistors0402:R_0R_0402") (at 91.44 96.52 270) (mirror x) (unit 1)
-    (in_bom no) (on_board yes) (dnp yes)
+    (in_bom yes) (on_board yes) (dnp yes)
     (property "Reference" "R801" (at 88.9 92.71 90)
       (effects (font (size 1.27 1.27) (thickness 0.15)) (justify right))
@@
       (effects (font (size 1.27 1.27) (thickness 0.15)) (justify left bottom) hide)
     )
-    (pin "SH1")
+    (pin "MP")
     (pin "1")
-    (pin "SH2")
     (pin "2")
     (instances
@@
   )
   (symbol (lib_id "antmicroResistors0402:R_10k_0402") (at 243.84 120.65 90) (unit 1)
-    (in_bom no) (on_board yes) (dnp yes)
+    (in_bom yes) (on_board yes) (dnp yes)
     (property "Reference" "R805" (at 245.11 116.84 90)
       (effects (font (size 1.27 1.27) (thickness 0.15)) (justify right))
@@
     (pin "3")
     (pin "4")
-    (pin "SH1")
-    (pin "SH2")
+    (pin "MP")
     (instances
       (project "cm4-baseboard"
