File: peripherals.kicad_sch (KiCad schematic)
At the start: 58 parts, among them J801 Socket_Samtec_ERF5_2x20_ERF5-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, J802 JST_SH_1x4_SM04B-SRSS-TB-LF-SN, J803 JST_SH_1x4_SM04B-SRSS-TB-LF-SN, J804 JST_SH_1x2_SM02B-SRSS-TB-LF-SN, U801 PN7160A1_VFQFN, Y801 Resonator_27.12MHz_XRCGB

Commit message: [#61534] Clean DNP properites
Other:
- moved on the sheet: C816, C824

Commit message: [#63565] Synchronize components with library, bump revision to 1.0.4
Other:
- company: Antmicro -> Antmicro Ltd
Changed lines of the file:
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@@
   (title_block
     (title "CM4 Baseboard")
-    (date "2024-06-19")
-    (rev "1.0.3")
-    (company "Antmicro")
+    (date "2024-08-02")
+    (rev "1.0.5")
+    (company "Antmicro Ltd")
     (comment 1 "www.antmicro.com")
   )
@@
     )
   )
-  (symbol (lib_id "antmicroFixedInductors:L_template_name") (at 309.88 107.95 0) (unit 1)
+  (symbol (lib_name "L_template_name_1") (lib_id "antmicroFixedInductors:L_template_name") (at 309.88 107.95 0) (unit 1)
     (in_bom no) (on_board yes) (dnp yes)
     (property "Reference" "L801" (at 312.42 105.41 0)

Commit message: [#65638] Post review fixes
Parts:
- L801, L802: footprint antmicro-footprints:L_0603_1608Metric -> antmicro-footprints:
Changed lines of the file:
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@@
   (title_block
     (title "CM4 Baseboard")
-    (date "2024-09-12")
+    (date "2024-09-13")
     (rev "1.0.5")
     (company "Antmicro Ltd")
@@
       (effects (font (size 1.27 1.27) (thickness 0.15)) (justify left bottom) hide)
     )
-    (property "Footprint" "antmicro-footprints:L_0603_1608Metric" (at 323.85 130.81 0)
+    (property "Footprint" "antmicro-footprints:" (at 323.85 130.81 0)
       (effects (font (size 1.27 1.27) (thickness 0.15)) (justify left bottom) hide)
     )
@@
     )
   )
-  (symbol (lib_name "L_template_name_1") (lib_id "antmicroFixedInductors:L_template_name") (at 309.88 107.95 0) (unit 1)
+  (symbol (lib_id "antmicroFixedInductors:L_template_name") (at 309.88 107.95 0) (unit 1)
     (in_bom no) (on_board yes) (dnp yes)
     (property "Reference" "L801" (at 312.42 105.41 0)
@@
       (effects (font (size 1.27 1.27) (thickness 0.15)) (justify left bottom) hide)
     )
-    (property "Footprint" "antmicro-footprints:L_0603_1608Metric" (at 323.85 115.57 0)
+    (property "Footprint" "antmicro-footprints:" (at 323.85 115.57 0)
       (effects (font (size 1.27 1.27) (thickness 0.15)) (justify left bottom) hide)
     )
